File: kicad/segments-2-the-absurd.kicad_pcb (KiCad board)
At the start: 2 copper layers, 35 parts, among them J1 Conn_01x02_Pin, J2 Conn_01x05_Socket, U1 STM32C011F6Px, U2 TM1637, U3 TM1637, U4 TM1637

Commit message: adding v-alpha prototype gerbers (note out of sync with kicad files)
Parts:
- removed C2: 4.7uF, Capacitor_SMD:C_0805_2012Metric
- removed C3: 100nF, Capacitor_SMD:C_0805_2012Metric
- added C17: 100nF, Capacitor_SMD:C_0603_1608Metric, B.Cu at (261.6, 113.5)
- added C18: 100pF, Capacitor_SMD:C_0603_1608Metric, B.Cu at (261.6, 111.8)
- added C19: 100pF, Capacitor_SMD:C_0603_1608Metric, B.Cu at (261.6, 109.2)
- added C20: 100uF, Capacitor_SMD:C_1206_3216Metric, B.Cu at (251.8, 154.7)
- added C21: 100nF, Capacitor_SMD:C_0603_1608Metric, B.Cu at (233.7, 172.7)
- added C22: 100pF, Capacitor_SMD:C_0603_1608Metric, B.Cu at (233.7, 169.7)
- added C23: 100pF, Capacitor_SMD:C_0603_1608Metric, B.Cu at (233.7, 167.4)
- added C24: 100nF, Capacitor_SMD:C_0603_1608Metric, B.Cu at (227.3, 109.7)
- added C25: 4.7uF, Capacitor_SMD:C_0603_1608Metric, B.Cu at (227.3, 111.5)
- added C26: 100nF, Capacitor_SMD:C_0603_1608Metric, B.Cu at (248.7, 116.8)
- added C27: 100nF, Capacitor_SMD:C_0603_1608Metric, B.Cu at (230.9, 115.1)
- added C28: 100nF, Capacitor_SMD:C_0603_1608Metric, B.Cu at (226.7, 113.3)
- added C29: 100nF, Capacitor_SMD:C_0603_1608Metric, B.Cu at (220.7, 145.7)
- added C30: 4.7uF, Capacitor_SMD:C_0603_1608Metric, B.Cu at (220.7, 147.2)
- added C31: 100nF, Capacitor_SMD:C_0603_1608Metric, B.Cu at (243.7, 156.8)
- added C32: 100nF, Capacitor_SMD:C_0603_1608Metric, B.Cu at (211.6, 157.2)
- added C33: 100nF, Capacitor_SMD:C_0603_1608Metric, B.Cu at (209.0, 157.2)
- added C34: 100uF, Capacitor_SMD:C_1206_3216Metric, B.Cu at (233.8, 174.6)
- added C35: 100nF, Capacitor_SMD:C_0603_1608Metric, B.Cu at (252.2, 151.9)
- added C36: 100pF, Capacitor_SMD:C_0603_1608Metric, B.Cu at (252.2, 150.4)
- added C37: 100pF, Capacitor_SMD:C_0603_1608Metric, B.Cu at (252.2, 148.1)
- added C38: 100uF, Capacitor_SMD:C_1206_3216Metric, B.Cu at (309.8, 136.0)
- added C39: 100nF, Capacitor_SMD:C_0603_1608Metric, B.Cu at (310.5, 134.1)
- added C40: 100pF, Capacitor_SMD:C_0603_1608Metric, B.Cu at (310.5, 130.9)
- added C41: 100pF, Capacitor_SMD:C_0603_1608Metric, B.Cu at (310.5, 128.8)
- added C42: 100uF, Capacitor_SMD:C_1206_3216Metric, B.Cu at (309.5, 174.4)
- added C43: 100nF, Capacitor_SMD:C_0603_1608Metric, B.Cu at (310.1, 172.5)
- added C44: 100pF, Capacitor_SMD:C_0603_1608Metric, B.Cu at (310.1, 169.4)
- added C45: 100pF, Capacitor_SMD:C_0603_1608Metric, B.Cu at (310.1, 167.4)
- added D10: SP410561N, 01-User-Footprints:7-Seg-3D_CA_ARKLED_SP410561N, F.Cu at (261.6, 150.9)
- added D11: SP410561N, 01-User-Footprints:7-Seg-3D_CA_ARKLED_SP410561N, F.Cu at (299.7, 150.9)
- added D12: SP410561N, 01-User-Footprints:7-Seg-3D_CA_ARKLED_SP410561N, F.Cu at (337.8, 150.9)
- added D13: SP410561N, 01-User-Footprints:7-Seg-3D_CA_ARKLED_SP410561N, F.Cu at (223.5, 170.4)
- added D14: SP410561N, 01-User-Footprints:7-Seg-3D_CA_ARKLED_SP410561N, F.Cu at (261.6, 170.4)
- added D15: SP410561N, 01-User-Footprints:7-Seg-3D_CA_ARKLED_SP410561N, F.Cu at (299.7, 170.4)
- added D16: SP410561N, 01-User-Footprints:7-Seg-3D_CA_ARKLED_SP410561N, F.Cu at (337.8, 170.4)
- added D7: SP410561N, 01-User-Footprints:7-Seg-3D_CA_ARKLED_SP410561N, F.Cu at (299.7, 131.3)
- added D8: SP410561N, 01-User-Footprints:7-Seg-3D_CA_ARKLED_SP410561N, F.Cu at (337.8, 131.3)
- added D9: SP410561N, 01-User-Footprints:7-Seg-3D_CA_ARKLED_SP410561N, F.Cu at (223.5, 150.9)
- added J10: Conn_01x02_Pin, Connector_PinHeader_2.54mm:PinHeader_1x02_P2.54mm_Vertical, B.Cu at (306.2, 146.3)
- added J11: Conn_01x02_Pin, Connector_PinHeader_2.54mm:PinHeader_1x02_P2.54mm_Vertical, B.Cu at (238.8, 123.2)
- added J12: Conn_01x02_Pin, Connector_PinHeader_2.54mm:PinHeader_1x02_P2.54mm_Vertical, B.Cu at (249.7, 105.9)
- added J13: Conn_01x02_Pin, Connector_PinHeader_2.54mm:PinHeader_1x02_P2.54mm_Vertical, B.Cu at (228.3, 168.0)
- added J14: Conn_01x02_Pin, Connector_PinHeader_2.54mm:PinHeader_1x02_P2.54mm_Vertical, B.Cu at (244.3, 144.3)
- added J15: Conn_01x02_Pin, Connector_PinHeader_2.54mm:PinHeader_1x02_P2.54mm_Vertical, B.Cu at (304.8, 128.9)
- added J16: Conn_01x02_Pin, Connector_PinHeader_2.54mm:PinHeader_1x02_P2.54mm_Vertical, B.Cu at (305.1, 169.0)
- added J17: Conn_01x02_Pin, Connector_PinHeader_2.54mm:PinHeader_1x02_P2.54mm_Vertical, B.Cu at (236.0, 131.7)
- added J18: Conn_01x03_Pin, Connector_PinHeader_1.27mm:PinHeader_1x03_P1.27mm_Vertical, B.Cu at (214.9, 113.3)
- added J19: Conn_01x03_Pin, Connector_PinHeader_1.27mm:PinHeader_1x03_P1.27mm_Vertical, B.Cu at (208.0, 143.5)
- added J20: Conn_01x02_Pin, Connector_PinHeader_2.54mm:PinHeader_1x02_P2.54mm_Vertical, B.Cu at (232.9, 131.7)
- added J4: Conn_01x05_Socket, Connector_PinHeader_2.54mm:PinHeader_1x05_P2.54mm_Vertical, B.Cu at (218.2, 106.7)
- added J6: Conn_01x05_Socket, Connector_PinHeader_2.54mm:PinHeader_1x05_P2.54mm_Vertical, B.Cu at (207.8, 153.9)
- added J7: Conn_01x02_Pin, Connector_PinHeader_1.27mm:PinHeader_1x02_P1.27mm_Vertical, B.Cu at (214.6, 118.9)
- added J8: Conn_01x02_Pin, Connector_PinHeader_1.27mm:PinHeader_1x02_P1.27mm_Vertical, B.Cu at (208.0, 149.1)
- added J9: Conn_01x02_Pin, Connector_PinHeader_2.54mm:PinHeader_1x02_P2.54mm_Vertical, B.Cu at (304.8, 109.7)
- added JP1: Jumper_3_Bridged12, Jumper:SolderJumper-3_P1.3mm_Bridged12_RoundedPad1.0x1.5mm, B.Cu at (283.0, 125.7)
- added JP2: Jumper_3_Bridged12, Jumper:SolderJumper-3_P1.3mm_Bridged12_RoundedPad1.0x1.5mm, B.Cu at (283.1, 132.2)
- added R10: 10K, Resistor_SMD:R_0603_1608Metric, B.Cu at (243.1, 126.2)
- added R11: 10K, Resistor_SMD:R_0603_1608Metric, B.Cu at (260.7, 106.8)
- added R12: 10K, Resistor_SMD:R_0603_1608Metric, B.Cu at (262.5, 106.8)
- added R13: 10K, Resistor_SMD:R_0603_1608Metric, B.Cu at (232.9, 164.8)
- added R14: 10K, Resistor_SMD:R_0603_1608Metric, B.Cu at (234.4, 164.8)
- added R15: 10K, Resistor_SMD:R_0603_1608Metric, B.Cu at (229.9, 113.5)
- added R16: 10K, Resistor_SMD:R_0603_1608Metric, B.Cu at (223.5, 148.8)
- added R17: 10K, Resistor_SMD:R_0603_1608Metric, B.Cu at (251.5, 145.8)
- added R18: 10K, Resistor_SMD:R_0603_1608Metric, B.Cu at (253.0, 145.8)
- added R19: 10K, Resistor_SMD:R_0603_1608Metric, B.Cu at (309.8, 126.5)
- added R20: 10K, Resistor_SMD:R_0603_1608Metric, B.Cu at (311.3, 126.5)
- added R21: 10K, Resistor_SMD:R_0603_1608Metric, B.Cu at (309.4, 165.1)
- added R22: 10K, Resistor_SMD:R_0603_1608Metric, B.Cu at (310.9, 165.1)
- added R8: 10K, Resistor_SMD:R_0603_1608Metric, B.Cu at (311.4, 145.8)
- added R9: 10K, Resistor_SMD:R_0603_1608Metric, B.Cu at (241.6, 126.2)
- added REF**: MountingHole_3mm, MountingHole:MountingHole_3mm, F.Cu at (340.4, 113.3)
- added REF**: MountingHole_3mm, MountingHole:MountingHole_3mm, F.Cu at (343.2, 171.0)
- added REF**: MountingHole_3mm, MountingHole:MountingHole_3mm, F.Cu at (217.9, 168.7)
- added REF**: MountingHole_3mm, MountingHole:MountingHole_3mm, F.Cu at (215.9, 91.2)
- added U10: STM32C011F6Px, Package_SO:TSSOP-20_4.4x6.5mm_P0.65mm, B.Cu at (214.6, 148.3)
- added U11: TM1637, 01-User-Footprints:TM_TM1637(TA2007)_SOC-20_12.6x7.5_P1.27_PD0.44x2, B.Cu at (260.6, 151.0)
- added U12: TM1637, 01-User-Footprints:TM_TM1637(TA2007)_SOC-20_12.6x7.5_P1.27_PD0.44x2, B.Cu at (318.8, 131.8)
- added U13: TM1637, 01-User-Footprints:TM_TM1637(TA2007)_SOC-20_12.6x7.5_P1.27_PD0.44x2, B.Cu at (318.8, 170.7)
- added U5: TM1637, 01-User-Footprints:TM_TM1637(TA2007)_SOC-20_12.6x7.5_P1.27_PD0.44x2, B.Cu at (271.0, 112.0)
- added U6: TM1637, 01-User-Footprints:TM_TM1637(TA2007)_SOC-20_12.6x7.5_P1.27_PD0.44x2, B.Cu at (242.2, 170.7)
- added U7: TXS0108E, Package_SO:TSSOP-20_4.4x6.5mm_P0.65mm, B.Cu at (248.7, 112.2)
- added U8: STM32C011F6Px, Package_SO:TSSOP-20_4.4x6.5mm_P0.65mm, B.Cu at (220.5, 113.8)
- added U9: TXS0108E, Package_SO:TSSOP-20_4.4x6.5mm_P0.65mm, B.Cu at (242.6, 151.6)
- C1, C11, C15, C7: footprint Capacitor_SMD:C_0805_2012Metric -> Capacitor_SMD:C_0603_1608Metric; moved to B.Cu
- C10, C14, C6: value 100nF -> 100pF; footprint Capacitor_SMD:C_0805_2012Metric -> Capacitor_SMD:C_0603_1608Metric; moved to B.Cu
- C12, C16, C8: value 100pF -> 100uF; footprint Capacitor_SMD:C_0805_2012Metric -> Capacitor_SMD:C_1206_3216Metric; moved to B.Cu
- C13, C5, C9: value 100u -> 100nF; footprint Capacitor_SMD:C_0805_2012Metric -> Capacitor_SMD:C_0603_1608Metric; moved to B.Cu
- C4: value 100nF -> 100uF; footprint Capacitor_SMD:C_0805_2012Metric -> Capacitor_SMD:C_1206_3216Metric; moved to B.Cu
- J1: value Conn_01x02_Pin -> Conn_01x03_Pin; footprint Connector_PinHeader_1.27mm:PinHeader_1x02_P1.27mm_Vertical -> 01-User-Footprints:Power-Conn-3P-D0.65-P5-BD7.8x15
- J2: value Conn_01x05_Socket -> Conn_01x08_Pin; footprint Connector_PinHeader_1.27mm:PinHeader_1x05_P1.27mm_Vertical -> Connector_PinHeader_2.54mm:PinHeader_1x08_P2.54mm_Vertical; moved to B.Cu
- R1, R2, R3, R4, R5, R6, R7: footprint Resistor_SMD:R_0805_2012Metric -> Resistor_SMD:R_0603_1608Metric; moved to B.Cu
- U1: value STM32C011F6Px -> 74HC595; footprint Package_SO:TSSOP-20_4.4x6.5mm_P0.65mm -> Package_SO:SOP-16_3.9x9.9mm_P1.27mm; moved to B.Cu
- U2, U3, U4: footprint 01-User-Footprints:TM_TM1637(TA2007)_SOC20 -> 01-User-Footprints:TM_TM1637(TA2007)_SOC-20_12.6x7.5_P1.27_PD0.44x2; moved to B.Cu
- moved C8 204.8 mm to (309.7, 155.4), turned to 180 degrees
- moved C4 203.7 mm to (309.2, 117.2), turned to 180 degrees
- moved C5 195.9 mm to (309.9, 115.3), turned to 180 degrees
- moved C6 193.5 mm to (309.9, 112.3), turned to 180 degrees
- moved C7 185.5 mm to (309.9, 110.2), turned to 180 degrees
- moved U2 177.3 mm to (318.8, 113.2)
- moved U3 175.3 mm to (318.8, 151.6)
- moved C11 158.6 mm to (310.5, 148.1), turned to 180 degrees
- moved C9 151.4 mm to (310.5, 153.5), turned to 180 degrees
- moved C10 149.2 mm to (310.5, 150.4), turned to 180 degrees
- moved R5 142.1 mm to (309.1, 107.7), turned to -90 degrees
- moved R6 132.9 mm to (310.6, 107.7), turned to -90 degrees
- moved R7 132.7 mm to (309.8, 145.8), turned to -90 degrees
- moved R2 125.7 mm to (226.3, 128.4), turned to 180 degrees
- moved R3 125.1 mm to (226.4, 130.4), turned to 180 degrees
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Connections:
- C1 pad 1: VDD -> GND
- C1 pad 2: GND -> +3V3
- C10 pad 1: VDD -> /S2A_Serf2/B_DAT
- C11 pad 1: /B_DAT -> /S2A_Serf2/B_CLK
- C12 pad 1: /B_CLK -> /S2A_Serf1/V_DRIVER
- C13 pad 1: VDD -> /S2A_Serf1/V_DRIVER
- C14 pad 1: VDD -> /S2A_Serf1/C_DAT
- C15 pad 1: /C_DAT -> /S2A_Serf1/C_CLK
- C16 pad 1: /C_CLK -> /S2A_Serf1/V_DRIVER
- C4 pad 1: GND -> /S2A_Serf1/V_DRIVER
- C4 pad 2: VDD -> GND
- C5 pad 1: VDD -> /S2A_Serf1/V_DRIVER
- C6 pad 1: VDD -> /S2A_Serf1/B_DAT
- C7 pad 1: /A_DAT -> /S2A_Serf1/B_CLK
- C8 pad 1: /A_CLK -> /S2A_Serf2/V_DRIVER
- C9 pad 1: VDD -> /S2A_Serf2/V_DRIVER
- J1 pad 1: /nRESET -> +3V3
- J2 pad 1: VDD -> /DISP_EN
- J2 pad 2: /SWDIO -> /SPI_SCK
- J2 pad 3: /SWCLK_BOOT0 -> /SPI_MISO
- J2 pad 4: /nRESET -> /SPI_MOSI
- J2 pad 5: GND -> /nRESET_ALL
- R1 pad 1: VDD -> +3V3
- R1 pad 2: /nRESET -> /SPI_NSS1
- R2 pad 1: VDD -> +3V3
- R2 pad 2: /A_DAT -> /SPI_NSS2
- R3 pad 1: VDD -> +3V3
- R3 pad 2: /A_CLK -> /nSS_nOE
- R4 pad 1: VDD -> +3V3
- R4 pad 2: /B_DAT -> Net-(U1-~{SRCLR})
- R5 pad 1: VDD -> /S2A_Serf1/V_DRIVER
- R5 pad 2: /B_CLK -> /S2A_Serf1/B_DAT
- R6 pad 1: VDD -> /S2A_Serf1/V_DRIVER
- R6 pad 2: /C_DAT -> /S2A_Serf1/B_CLK
- R7 pad 1: VDD -> /S2A_Serf2/V_DRIVER
- R7 pad 2: /C_CLK -> /S2A_Serf2/B_DAT
- U1 pad 1: unconnected-(U1-PB7-Pad1) -> /SPI_NSS2
- U1 pad 10: unconnected-(U1-PA3-Pad10) -> Net-(U1-~{SRCLR})
- U1 pad 11: /SPI1-NSS -> /nSS_CLK
- U1 pad 12: /SPI1-SCK -> /nSS_CLK
- U1 pad 13: /SPI1-MISO_DOUT -> /nSS_nOE
- U1 pad 14: /SPI1-MOSI_DIN -> /nSS_SDA
- U1 pad 15: /B_DAT -> /SPI_NSS1
- U1 pad 16: /C_CLK -> +3V3
- U1 pad 2: /OSC-IN -> unconnected-(U1-QC-Pad2)
- U1 pad 3: /OSC-OUT -> unconnected-(U1-QD-Pad3)
- U1 pad 4: VDD -> unconnected-(U1-QE-Pad4)
- U1 pad 5: GND -> unconnected-(U1-QF-Pad5)
- U1 pad 6: /nRESET -> unconnected-(U1-QG-Pad6)
- U1 pad 7: /A_CLK -> unconnected-(U1-QH-Pad7)
- U1 pad 8: /A_DAT -> GND
- U1 pad 9: /B_CLK -> unconnected-(U1-QH'-Pad9)
- U2 pad 10: Net-(D2-DIG3) -> Net-(D4-DIG3)
- U2 pad 11: Net-(D2-DIG2) -> Net-(D4-DIG2)
- U2 pad 12: Net-(D2-DIG1) -> Net-(D4-DIG1)
- U2 pad 13: Net-(D1-DIG3) -> Net-(D3-DIG3)
- U2 pad 14: Net-(D1-DIG2) -> Net-(D3-DIG2)
- U2 pad 15: Net-(D1-DIG1) -> Net-(D3-DIG1)
- U2 pad 16: VDD -> /S2A_Serf1/V_DRIVER
- U2 pad 17: /A_DAT -> /S2A_Serf1/B_DAT
- U2 pad 18: /A_CLK -> /S2A_Serf1/B_CLK
- U2 pad 2: Net-(D1-a) -> Net-(D3-a)
- U2 pad 3: Net-(D1-b) -> Net-(D3-b)
- U2 pad 4: Net-(D1-c) -> Net-(D3-c)
- U2 pad 5: Net-(D1-d) -> Net-(D3-d)
- U2 pad 6: Net-(D1-e) -> Net-(D3-e)
- U2 pad 7: Net-(D1-f) -> Net-(D3-f)
- U2 pad 8: Net-(D1-g) -> Net-(D3-g)
- U2 pad 9: Net-(D1-DPX) -> Net-(D3-DPX)
- U3 pad 10: Net-(D4-DIG3) -> Net-(D12-DIG3)
- U3 pad 11: Net-(D4-DIG2) -> Net-(D12-DIG2)
- U3 pad 12: Net-(D4-DIG1) -> Net-(D12-DIG1)
- U3 pad 13: Net-(D3-DIG3) -> Net-(D11-DIG3)
- U3 pad 14: Net-(D3-DIG2) -> Net-(D11-DIG2)
- U3 pad 15: Net-(D3-DIG1) -> Net-(D11-DIG1)
- U3 pad 16: VDD -> /S2A_Serf2/V_DRIVER
- U3 pad 17: /B_DAT -> /S2A_Serf2/B_DAT
- U3 pad 18: /B_CLK -> /S2A_Serf2/B_CLK
- U3 pad 2: Net-(D3-a) -> Net-(D11-a)
- U3 pad 3: Net-(D3-b) -> Net-(D11-b)
- U3 pad 4: Net-(D3-c) -> Net-(D11-c)
- U3 pad 5: Net-(D3-d) -> Net-(D11-d)
- U3 pad 6: Net-(D3-e) -> Net-(D11-e)
- U3 pad 7: Net-(D3-f) -> Net-(D11-f)
- U3 pad 8: Net-(D3-g) -> Net-(D11-g)
- U3 pad 9: Net-(D3-DPX) -> Net-(D11-DPX)
- U4 pad 16: VDD -> /S2A_Serf1/V_DRIVER
- U4 pad 17: /C_DAT -> /S2A_Serf1/C_DAT
- U4 pad 18: /C_CLK -> /S2A_Serf1/C_CLK
Routing:
- net /S2A_Serf2/V_DRIVER: track 0.00 -> 263.7 mm, vias 0 -> 2
- net GND: track 0.00 -> 258.7 mm, vias 0 -> 62
- net /S2A_Serf1/V_DRIVER: track 0.00 -> 200.4 mm
- net +3V3: track 0.00 -> 141.1 mm, vias 0 -> 28
- net +5V: track 0.00 -> 128.4 mm, vias 0 -> 3
- net /nRESET_ALL: track 0.00 -> 116.5 mm, vias 0 -> 6
- net /S2A_Serf2/D_DAT: track 0.00 -> 85.4 mm, vias 0 -> 2
- net /S2A_Serf2/B_CLK: track 0.00 -> 84.1 mm, vias 0 -> 4
- net /S2A_Serf1/B_DAT: track 0.00 -> 82.0 mm, vias 0 -> 2
- net /S2A_Serf2/D_CLK: track 0.00 -> 81.5 mm, vias 0 -> 2
- net /S2A_Serf2/B_DAT: track 0.00 -> 80.0 mm, vias 0 -> 4
- net Net-(D1-d): track 0.00 -> 79.1 mm, vias 0 -> 2
- net /S2A_Serf1/D_DAT: track 0.00 -> 77.8 mm, vias 0 -> 3
- net /S2A_Serf1/D_CLK: track 0.00 -> 76.3 mm, vias 0 -> 2
- net /S2A_Serf1/B_CLK: track 0.00 -> 72.5 mm, vias 0 -> 2
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- added copper zone on B.Cu, net +3V3
- added copper zone on F.Cu, net GND
Other:
- board outline added: 154.2 x 81.6 mm
- board text added: "!! SET VOLTAGE !!"
- board text added: "5V"
- board text added: "CLK"
- board text added: "DE"
- board text added: "DEBUG1"
- board text added: "DEBUG2"
- board text added: "I2C"
- board text added: "MISO"
- board text added: "MOSI"
- board text added: "NRST"
- board text added: "NSS1"
- board text added: "NSS2"
- board text added: "POWER"
- board text added: "SCK"
- board text added: "SCLK"
- board text added: "SDA"
- board text added: "SER"
- board text added: "SI"
- board text added: "SO"
- board text added: "SPI"
- board text added: "SPI_MISO"
- board text added: "SPI_MOSI"
- board text added: "SPI_SCK"
- board text added: "SPI_SR"
- board text added: "SR_CLK"
- board text added: "SR_SDA"
- board text added: "SR_nOE"
- board text added: "V_DRIVER1"
- board text added: "V_DRIVER2"
- board text added: "~{SS1}"
- board text added: "~{SS2}"
- board text removed: "DEBUG"
- board text removed: "Driver A"
- board text removed: "Driver B"
- board text removed: "Driver C"
- board text removed: "SWCLK"
- board text removed: "Short for Reset"
