File: kicad/segments-2-the-absurd.kicad_sch (KiCad schematic)
At the start: 15 parts, among them J1 Conn_01x08_Pin, J6 Conn_01x03_Pin, U1 74HC595, Y1 Crystal

Commit message: adding v-alpha prototype gerbers (note out of sync with kicad files)
Parts:
- removed TP1, TP2, TP3, TP4: TestPoint, symbol Connector:TestPoint
- added J17, J20: Conn_01x02_Pin, Connector_PinHeader_2.54mm:PinHeader_1x02_P2.54mm_Vertical, symbol Connector:Conn_01x02_Pin
- C1: value 0.1u -> 100nF; footprint (none) -> Capacitor_SMD:C_0603_1608Metric; Basic/Extended (none) -> Basic; DOUBLE_CHECK (none) -> x; JLPCB_MPN (none) -> CC0603KRX7R9BB104; JLPCB_Mfg (none) -> YAGEO; JLPCB_Part_No (none) -> C14663; JLPCB_Price (none) -> 0.0021; JLPCB_URL (none) -> https://jlcpcb.com/partdetail/Yageo-CC0603KRX7R9BB104/C14663; LCSC Part # (none) -> C14663
- C2, C3: footprint Capacitor_SMD:C_0805_2012Metric -> Capacitor_SMD:C_0603_1608Metric; Basic/Extended (none) -> Basic; DOUBLE_CHECK (none) -> x; JLPCB_MPN (none) -> CL10C200JB8NNNC; JLPCB_Mfg (none) -> Samsung Electro-Mechanics; JLPCB_Part_No (none) -> C1648; JLPCB_Price (none) -> 0.005; JLPCB_URL (none) -> https://jlcpcb.com/partdetail/2000-CL10C200JB8NNNC/C1648; LCSC Part # (none) -> C1648
- J1: renamed from J6; footprint (none) -> 01-User-Footprints:Power-Conn-3P-D0.65-P5-BD7.8x15; Basic/Extended (none) -> Extended; DNP (none) -> DNP; JLPCB_MPN (none) -> XY126V-5.0-3P; JLPCB_Mfg (none) -> Ningbo Xinlaiya Elec.; JLPCB_Part_No (none) -> C557647; JLPCB_URL (none) -> https://jlcpcb.com/partdetail/Ningbo_Xinlaiya_elec-XY126V_5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; LCSC Part # (none) -> C557647; now not fitted; now left out of the parts list
- J2: renamed from J1; footprint (none) -> Connector_PinHeader_2.54mm:PinHeader_1x08_P2.54mm_Vertical; DNP (none) -> DNP
- R1, R2, R3, R4: footprint (none) -> Resistor_SMD:R_0603_1608Metric; Basic/Extended (none) -> Basic; JLPCB_MPN (none) -> 0603WAF1002T5E; JLPCB_Mfg (none) -> UNI-ROYAL(Uniroyal Elec); JLPCB_Part_No (none) -> C25804; JLPCB_URL (none) -> https://jlcpcb.com/partdetail/26547-0603WAF1002T5E/C25804; LCSC Part # (none) -> C25804
- U1: footprint (none) -> Package_SO:SOP-16_3.9x9.9mm_P1.27mm; Basic/Extended (none) -> Extended; DOUBLE_CHECK (none) -> done, 3.9x9.9; DOUBLE_CHECK_SYMB (none) -> done; JLCPN C110383 -> C5451631; JLCPrice 0.14 -> .06; JLCUrl https://jlcpcb.com/partdetail/Shenzhen_FumanElec-74HC595A/C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 -> https://jlcpcb.com/partdetail/HxyMosfet-74HC595D/C5451631?_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; JLPCB_MPN 74HC595 -> 74HC595D; JLPCB_Part_No (none) -> C5451631; JLPCB_Price (none) -> .06; JLPCB_URL (none) -> https://jlcpcb.com/partdetail/HxyMosfet-74HC595D/C5451631?_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; LCSC Part # (none) -> C5451631
- Y1: DNP (none) -> DNP; JLPCB_URL (none) -> https://www.lcsc.com/product-detail/Crystals_Seiko-Epson-Q1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
Connections:
- net +3V3: now also J1.1 (Pin_1); no longer J1.2 (Pin_2)
- net GND: now also J1.2 (Pin_2); no longer J1.1 (Pin_1)
- net nSS_CLK: now also J17.2 (Pin_2)
- net nSS_SDA: now also J17.1 (Pin_1)
- net S2A_Serf1/nSS renamed SPI_NSS1
- net SPI_NSS1: now also J20.1 (Pin_1); no longer R2.2, U1.1 (QB)
- new net SPI_NSS2: J20.2 (Pin_2), R2.2, U1.1 (QB)
Other:
- note added: "ADD USER INTERFACE BUTTON ?"
- note added: "Test Points"
- note removed: "=== TODOs === [x] test points [ ] level shifter"
